Commit message: added files for ros2_control in simulation

File: urdf/camera.xacro (robot description, xacro)
@@ -4,5 +4,5 @@
         <parent link="chassis"/>
         <child link="camera_link"/>
-        <origin xyz="0.305 0 0.08" rpy="0 0 0"/>
+        <origin xyz="0.215 0 0.08" rpy="0 0 0"/>
     </joint>
     <link name="camera_link">

File: urdf/myrobot.urdf.xacro (robot description, xacro)
@@ -1,6 +1,12 @@
 <?xml version="1.0"?>
 <robot xmlns:xacro="http://www.ros.org/wiki/xacro" name="Robot">
+	<xacro:arg name="use_ros2_control" default="true" />
 	<xacro:include filename="robot_core.xacro" />
-	<xacro:include filename="gazebo_control.xacro" />
+	<xacro:if value="$(arg use_ros2_control)">
+		<xacro:include filename="ros2_control.xacro" />
+	</xacro:if>
+	<xacro:unless value="$(arg use_ros2_control)">
+		<xacro:include filename="gazebo_control.xacro" />
+	</xacro:unless>
 	<xacro:include filename="camera.xacro" />
 </robot>

File: urdf/robot_core.xacro (robot description, xacro)
@@ -2,4 +2,32 @@
 <robot xmlns:xacro="http://www.ros.org/wiki/xacro">
 	<xacro:include filename="inertial_macros.xacro" />
+	<!-- <xacro:property name="chassis_length" value="0.335"/>
+    <xacro:property name="chassis_width" value="0.265"/>
+    <xacro:property name="chassis_height" value="0.138"/>
+    <xacro:property name="chassis_mass" value="1.0"/>
+    <xacro:property name="wheel_radius" value="0.034"/>
+    <xacro:property name="wheel_thickness" value="0.026"/>
+    <xacro:property name="wheel_mass" value="0.05"/>
+    <xacro:property name="wheel_offset_x" value="0.226"/>
+    <xacro:property name="wheel_offset_y" value="0.166"/>
+    <xacro:property name="wheel_offset_z" value="0.01"/>
+    <xacro:property name="caster_wheel_radius" value="0.01"/>
+    <xacro:property name="caster_wheel_mass" value="0.01"/>
+    <xacro:property name="caster_wheel_offset_x" value="0.075"/>
+    <xacro:property name="caster_wheel_offset_z" value="${wheel_offset_z - wheel_radius + caster_wheel_radius}"/> -->
+	<xacro:property name="chassis_length" value="0.21"/>
+    <xacro:property name="chassis_width" value="0.2"/>
+    <xacro:property name="chassis_height" value="0.08"/>
+    <xacro:property name="chassis_mass" value="1.0"/>
+    <xacro:property name="wheel_radius" value="0.035"/>
+    <xacro:property name="wheel_thickness" value="0.018"/>
+    <xacro:property name="wheel_mass" value="0.1"/>
+    <xacro:property name="wheel_offset_x" value="0.179"/>
+    <xacro:property name="wheel_offset_y" value="0.13"/>
+    <xacro:property name="wheel_offset_z" value="0.01"/>
+    <xacro:property name="caster_wheel_radius" value="0.01"/>
+    <xacro:property name="caster_wheel_mass" value="0.01"/>
+    <xacro:property name="caster_wheel_offset_x" value="0.085"/>
+    <xacro:property name="caster_wheel_offset_z" value="${wheel_offset_z - wheel_radius + caster_wheel_radius}"/>
 	<material name="white">
     <color rgba="1 1 1 1"/>
@@ -24,24 +52,24 @@
 	    <parent link="base_link"/>
 	    <child link="chassis"/>
-	    <origin xyz="-0.1 0 0"/>
+	    <origin xyz="${-wheel_offset_x} 0 ${-wheel_offset_z}"/>
 	</joint>
 	<link name="chassis">
 		<!-- Visual and collision here -->
 	    <visual>
-	        <origin xyz="0.15 0 0.075" rpy="0 0 0"/>
+	        <origin xyz="${chassis_length/2} 0 ${chassis_height/2}"/>
 	        <geometry>
-	            <box size="0.3 0.3 0.15"/>
+	            <box size="${chassis_length} ${chassis_width} ${chassis_height}"/>
 	        </geometry>
 	        <material name="white"/>
 	    </visual>
 		<collision>
-			<origin xyz="0.15 0 0.075" rpy="0 0 0"/>
+			<origin xyz="${chassis_length/2} 0 ${chassis_height/2}"/>
 	        <geometry>
-	            <box size="0.3 0.3 0.15"/>
+	            <box size="${chassis_length} ${chassis_width} ${chassis_height}"/>
 	        </geometry>
 		</collision>
 		<!-- Inertial here -->
-		<xacro:inertial_box mass="0.5" x="0.3" y="0.3" z="0.15">
-			<origin xyz="0.15 0 0.075" rpy="0 0 0"/>
+		<xacro:inertial_box mass="0.5" x="${chassis_length}" y="${chassis_width}" z="${chassis_height}">
+			<origin xyz="${chassis_length/2} 0 ${chassis_height/2}" rpy="0 0 0"/>
 		</xacro:inertial_box>
 	</link>
@@ -53,5 +81,5 @@
 		<parent link="base_link"/>
 		<child link="left_wheel"/>
-		<origin xyz="0 0.175 0" rpy="-${pi/2} 0 0"/>
+		<origin xyz="0 ${wheel_offset_y} 0" rpy="-${pi/2} 0 0"/>
 		<axis xyz="0 0 1"/>
 	</joint>
@@ -59,5 +87,5 @@
 		<visual>
 			<geometry>
-				<cylinder radius="0.05" length="0.04"/>
+				<cylinder radius="${wheel_radius}" length="${wheel_thickness}"/>
 			</geometry>
 			<material name="blue"/>
@@ -65,8 +93,8 @@
 		<collision>
 			<geometry>
-				<cylinder radius="0.05" length="0.04"/>
+				<sphere radius="${wheel_radius}"/>
 			</geometry>
 		</collision>
-		<xacro:inertial_cylinder mass="0.1" length="0.05" radius="0.05">
+		<xacro:inertial_cylinder mass="${wheel_mass}" length="${wheel_thickness}" radius="${wheel_radius}">
 			<origin xyz="0 0 0" rpy="0 0 0"/>
 		</xacro:inertial_cylinder>
@@ -79,5 +107,5 @@
 		<parent link="base_link"/>
 		<child link="right_wheel"/>
-		<origin xyz="0 -0.175 0" rpy="${pi/2} 0 0"/>
+		<origin xyz="0 ${-wheel_offset_y} 0" rpy="${pi/2} 0 0"/>
 		<axis xyz="0 0 -1"/>
 	</joint>
@@ -85,5 +113,5 @@
 		<visual>
 			<geometry>
-				<cylinder length="0.04" radius="0.05" />
+				<cylinder length="${wheel_thickness}" radius="${wheel_radius}" />
 			</geometry>
 			<material name="blue"/>
@@ -91,8 +119,8 @@
 		<collision>
 			<geometry>
-				<cylinder length="0.04" radius="0.05" />
+				<sphere radius="${wheel_radius}"/>
 			</geometry>
 		</collision>
-		<xacro:inertial_cylinder mass="0.1" length="0.05" radius="0.05">
+		<xacro:inertial_cylinder mass="${wheel_mass}" length="${wheel_thickness}" radius="${wheel_radius}">
 			<origin xyz="0 0 0" rpy="0 0 0"/>
 		</xacro:inertial_cylinder>
@@ -105,10 +133,10 @@
 		<parent link="chassis"/>
 		<child link="caster_wheel"/>
-		<origin xyz="0.24 0 0" rpy="0 0 0"/>
+		<origin xyz="${caster_wheel_offset_x} 0 ${caster_wheel_offset_z}" />
 	</joint>
 	<link name="caster_wheel">
 		<visual>
 			<geometry>
-				<sphere radius="0.05" />
+				<sphere radius="${caster_wheel_radius}" />
 			</geometry>
 			<material name="black"/>
@@ -116,8 +144,8 @@
 		<collision>
 			<geometry>
-				<sphere radius="0.05" />
+				<sphere radius="${caster_wheel_radius}" />
 			</geometry>
 		</collision>
-		<xacro:inertial_sphere mass="0.1" radius="0.05">
+		<xacro:inertial_sphere mass="${caster_wheel_mass}" radius="${caster_wheel_radius}">
 			<origin xyz="0 0 0" rpy="0 0 0"/>
 		</xacro:inertial_sphere>
